Commit message: FIX(gazeobo): Change version - noetic
change version melodic to noetic and excute gazebo launch

File: hongdo_ros_description/urdf/hongdo_ros.urdf.g2.xacro (robot description, xacro)
@@ -1,4 +1,4 @@
 <?xml version="1.0" ?>
-<robot name="omo_r1" xmlns:xacro="http://ros.org/wiki/xacro">
+<robot name="hongdo_ros" xmlns:xacro="http://ros.org/wiki/xacro">
   <xacro:include filename="$(find hongdo_ros_description)/urdf/common_properties.xacro"/>
   <link name="base_footprint"/>
@@ -141,5 +141,5 @@
       <origin xyz="0 0 0.0" rpy="0.0 0 0.0"/>
       <geometry>
-        <mesh filename="package://hongdo_ros_description/meshes/sensors/omo_r1_lidar.stl" scale="0.001 0.001 0.001"/>
+        <mesh filename="package://hongdo_ros_description/meshes/sensors/hongdo_ros_lidar.stl" scale="0.001 0.001 0.001"/>
       </geometry>
       <material name="dark"/>
@@ -148,5 +148,5 @@
       <origin xyz="0 0 0.0" rpy="0.0 0 0.0"/>
       <geometry>
-        <mesh filename="package://omo_r1_description/meshes/sensors/omo_r1_lidar.stl" scale="0.001 0.001 0.001"/>
+        <mesh filename="package://hongdo_ros_description/meshes/sensors/hongdo_ros_lidar.stl" scale="0.001 0.001 0.001"/>
       </geometry>
     </collision>
@@ -168,5 +168,5 @@
       <origin xyz="0 0 0.0" rpy="1.5758 0.0 1.5758"/>
       <geometry>
-        <mesh filename="package://omo_r1_description/meshes/sensors/omo_r1_camera.stl" scale="0.001 0.001 0.001"/>
+        <mesh filename="package://hongdo_ros_description/meshes/sensors/hongdo_ros_camera.stl" scale="0.001 0.001 0.001"/>
       </geometry>
       <material name="dark"/>
@@ -175,9 +175,9 @@
       <origin xyz="0 0 0.0" rpy="1.5758 0.0 1.5758"/>
       <geometry>
-        <mesh filename="package://omo_r1_description/meshes/sensors/omo_r1_camera.stl" scale="0.001 0.001 0.001"/>
+        <mesh filename="package://hongdo_ros_description/meshes/sensors/hongdo_ros_camera.stl" scale="0.001 0.001 0.001"/>
       </geometry>
     </collision>
   </link> -->
-  <joint name="camera_rgb_joint" type="fixed">
+  <!-- <joint name="camera_rgb_joint" type="fixed">
     <origin xyz="0.03 0.0 0.0" rpy="0 0 0"/>
     <parent link="camera_link"/>
@@ -190,4 +190,4 @@
     <child link="camera_rgb_optical_frame"/>
   </joint>
-  <link name="camera_rgb_optical_frame"/>
+  <link name="camera_rgb_optical_frame"/> -->
 </robot>

File: hongdo_ros_description/urdf/hongdo_ros.urdf.xacro (robot description, xacro)
@@ -12,5 +12,5 @@
       <origin xyz="0.097 0.276 0.19" rpy="3.14 0 -1.57"/>
       <geometry>
-        <mesh filename="package://hongdo_ros_description/meshes/bases/hongdo_ros_body.stl" scale="0.001 0.001 0.001"/>
+        <mesh filename="package://hongdo_ros_description/meshes/bases/hongdo_ros_movebody.stl" scale="0.001 0.001 0.001"/>
       </geometry>
       <material name="light_black"/>
@@ -19,5 +19,5 @@
       <origin xyz="0.097 0.276 0.19" rpy="3.14 0 -1.57"/>
       <geometry>
-        <mesh filename="package://hongdo_ros_description/meshes/bases/hongdo_ros_body.stl" scale="0.001 0.001 0.001"/>
+        <mesh filename="package://hongdo_ros_description/meshes/bases/hongdo_ros_movebody.stl" scale="0.001 0.001 0.001"/>
       </geometry>
     </collision>
@@ -137,5 +137,5 @@
     <origin xyz="0.06 0 0.230" rpy="0.0 0 3.14159"/>
   </joint>
-  <!-- <link name="base_scan">
+  <link name="base_scan">
     <visual>
       <origin xyz="0 0 0.0" rpy="0.0 0 0.0"/>
@@ -158,11 +158,11 @@
                izz="0.001" />
     </inertial>
-  </link> -->
-  <!-- <joint name="camera_joint" type="fixed">
+  </link>
+  <joint name="camera_joint" type="fixed">
     <origin xyz="0.07 0.0 0.63" rpy="0 0.7 0"/>
     <parent link="base_link"/>
     <child link="camera_link"/>
-  </joint> -->
-  <!-- <link name="camera_link">
+  </joint>
+  <link name="camera_link">
     <visual>
       <origin xyz="0 0 0.0" rpy="1.5758 0.0 1.5758"/>
@@ -178,16 +178,16 @@
       </geometry>
     </collision>
-  </link> -->
-  <!-- <joint name="camera_rgb_joint" type="fixed">
+  </link>
+  <joint name="camera_rgb_joint" type="fixed">
     <origin xyz="0.03 0.0 0.0" rpy="0 0 0"/>
     <parent link="camera_link"/>
     <child link="camera_rgb_frame"/>
   </joint>
-  <link name="camera_rgb_frame"/> -->
-  <!-- <joint name="camera_rgb_optical_joint" type="fixed">
+  <link name="camera_rgb_frame"/>
+  <joint name="camera_rgb_optical_joint" type="fixed">
     <origin xyz="0 0 0" rpy="-1.57 0 -1.57"/>
     <parent link="camera_rgb_frame"/>
     <child link="camera_rgb_optical_frame"/>
-  </joint> -->
-  <!-- <link name="camera_rgb_optical_frame"/> -->
+  </joint>
+  <link name="camera_rgb_optical_frame"/>
 </robot>

File: hongdo_ros_gazebo/sdf/hongdo_ros.gazebo.xacro (robot description, xacro)
@@ -1,5 +1,5 @@
 <?xml version="1.0"?>
-<robot name="omo_r1_sim" xmlns:xacro="http://ros.org/wiki/xacro">
-  <xacro:include filename="$(find omo_r1_description)/urdf/omo_r1.urdf.xacro"/>
+<robot name="hongdo_ros_sim" xmlns:xacro="http://ros.org/wiki/xacro">
+  <xacro:include filename="$(find hongdo_ros_description)/urdf/hongdo_ros.urdf.xacro"/>
   <xacro:arg name="laser_visual"  default="false"/>
   <xacro:arg name="camera_visual" default="false"/>
@@ -54,5 +54,5 @@
   </gazebo>
   <gazebo>
-    <plugin name="omo_r1_controller" filename="libgazebo_ros_diff_drive.so">
+    <plugin name="hongdo_ros_controller" filename="libgazebo_ros_diff_drive.so">
       <commandTopic>cmd_vel</commandTopic>
       <odometryTopic>odom</odometryTopic>
